Commit message: Sync local repository with GitHub

File: src/bumperbot_description/urdf/bumperbot.urdf.xacro (robot description, xacro)
@@ -9,4 +9,6 @@
   <!-- Include ros2_control Plugins -->
   <xacro:include filename="$(find bumperbot_description)/urdf/bumperbot_ros2_control.xacro" />
+  <!-- Include Camera Model -->
+  <xacro:include filename="$(find bumperbot_description)/urdf/bumperbot_camera.xacro" />
   <link name="base_footprint"/>
   <link name="base_link">
@@ -218,3 +220,9 @@
     <color rgba="0.3 0.3 0.3 1"/>
   </material>
+  <material name="red">
+    <color rgba="1 0 0 1"/>
+  </material>
+  <material name="orange">
+    <color rgba="1 0.3 0.1 1"/>
+  </material>
 </robot>

File: src/bumperbot_description/urdf/bumperbot_gazebo.xacro (robot description, xacro)
@@ -60,4 +60,5 @@
         <render_engine>ogre2</render_engine>
       </plugin>
+      <!-- Add Camera Plugin - Creeated differently - see config and launch-->
     </xacro:unless>
   </gazebo>

Commit message: start moving

File: src/bumperbot_description/urdf/bumperbot.urdf.xacro (robot description, xacro)
@@ -67,6 +67,5 @@
     <axis xyz="0 1 0" />
   </joint>
-  <link
-    name="wheel_left_link">
+  <link name="wheel_left_link">
     <inertial>
       <origin xyz="0 0.014 0" rpy="0 0 0" />

Commit message: ultrasonic and camera added

File: src/bumperbot_description/urdf/bumperbot.urdf.xacro (robot description, xacro)
@@ -192,5 +192,5 @@
         <mesh filename="package://bumperbot_description/meshes/laser_link.STL" />
       </geometry>
-      <material name="dark_grey"/>
+      <material name="blue"/>
     </visual>
     <collision>
@@ -201,9 +201,32 @@
     </collision>
   </link>
-  <joint name="laser_joint" type="fixed">
+   <joint name="laser_joint" type="fixed">
     <origin xyz="-0.0050526 -0.0023221 0.1208" rpy="0 0 3.14" />
     <parent link="base_link" />
     <child link="laser_link" />
     <axis xyz="0 0 0" />
+  </joint>
+  <link name="ultrasonic_sensor_link">
+    <visual>
+      <geometry>
+        <box size="0.02 0.02 0.01"/>  <!-- Small box to represent the sensor -->
+      </geometry>
+      <material name="red"/>
+    </visual>
+    <origin xyz="0.05 0 0.005" rpy="0 0 0"/>  <!-- Adjust position relative to robot -->
+    <collision>
+      <geometry>
+        <box size="0.02 0.020 0.010"/>
+      </geometry>
+    </collision>
+    <inertial>
+      <mass value="0.015"/>
+      <inertia ixx="0.001" ixy="0" ixz="0" iyy="0.001" iyz="0" izz="0.001"/>
+    </inertial>
+  </link>
+  <joint name="ultrasonic_sensor_joint" type="fixed">
+    <parent link="base_link"/>  <!-- Change to your robot's main body -->
+    <child link="ultrasonic_sensor_link"/>
+    <origin xyz="0.05 0 0.0015" rpy="0 0 0"/>  <!-- Adjust placement -->
   </joint>
   <material name="blue">
@@ -223,5 +246,8 @@
   </material>
   <material name="orange">
-    <color rgba="1 0.3 0.1 1"/>
+    <color rgba="1 0.647 0 1"/>
+  </material>
+  <material name="green">
+      <color rgba="0 1 0 1"/>
   </material>
 </robot>

File: src/bumperbot_description/urdf/bumperbot_camera.xacro (robot description, xacro)
@@ -11,5 +11,5 @@
                 <box size="0.010 0.03 0.03"/>
             </geometry>
-            <material name="orange"/>
+            <color rgba="1 0.647 0 1"/> <!-- Orange color -->
         </visual>
         <visual>
@@ -18,5 +18,5 @@
                 <cylinder radius="0.002" length="0.1"/>
             </geometry>
-            <material name="orange"/>
+            <color rgba="1 0.647 0 1"/> <!-- Orange color -->
         </visual>
     </link>
@@ -28,5 +28,5 @@
     <link name="camera_link_optical"></link>
     <gazebo reference="camera_link">
-        <material>Gazebo/Black</material>
+        <material>Gazebo/Orange</material>
         <sensor name="camera" type="camera">
             <pose> 0 0 0 0 0 0 </pose>

File: src/bumperbot_description/urdf/bumperbot_gazebo.xacro (robot description, xacro)
@@ -144,3 +144,41 @@
     </sensor>
   </gazebo>
+  <!-- HC-SR04 sensor-->
+    <gazebo reference="ultrasonic_sensor_link">
+    <sensor name="ultrasonic_sensor" type="gpu_lidar">
+      <always_on>true</always_on>
+      <visualize>true</visualize>
+      <topic>ultrasonic</topic>
+      <update_rate>50</update_rate> <!-- Matches typical HC-SR04 behavior -->
+      <pose>0.1 0 0.1 0 0 0</pose> <!-- Adjust pose relative to the link -->
+      <gz_frame_id>ultrasonic_sensor_link</gz_frame_id>
+      <lidar>
+        <scan>
+          <horizontal>
+            <samples>1</samples> <!-- Single ray for HC-SR04 -->
+            <resolution>1.0</resolution>
+            <min_angle>0.0</min_angle>
+            <max_angle>0.0</max_angle>
+          </horizontal>
+          <vertical>
+            <samples>1</samples>
+            <resolution>1.0</resolution>
+            <min_angle>0.0</min_angle>
+            <max_angle>0.0</max_angle>
+          </vertical>
+        </scan>
+        <range>
+          <min>0.02</min> <!-- Minimum range: 2 cm -->
+          <max>4.0</max> <!-- Maximum range: 400 cm -->
+          <resolution>0.003</resolution> <!-- Accuracy: ±3 mm -->
+        </range>
+        <noise>
+          <type>gaussian</type>
+          <mean>0.0</mean>
+          <stddev>0.003</stddev> <!-- Noise matches accuracy of ±3 mm -->
+        </noise>
+      </lidar>
+    </sensor>
+    <!-- No additional plugin needed since gz-sim-sensors-system is already included globally -->
+  </gazebo>
 </robot>
